File: CE2_LFO.sch (KiCad schematic (older format))
At the start: 21 parts, among them J1 TriangleOut, J2 SquareOut, SW1 SW_DPDT_x2, U1 TL074

Commit message: First commit
Connections:
- net 6V renamed VREF
Other:
- moved on the sheet: R10, R9, U1E
Changed lines of the file:
@@
 encoding utf-8
 Sheet 1 1
-Title ""
+Title "CE2_LFO"
 Date ""
-Rev ""
+Rev "v1.0"
 Comp ""
 Comment1 ""
@@
 L Amplifier_Operational:TL074 U1
 U 5 1 6286E596
-P 1600 5300
-F 0 "U1" H 1558 5346 50  0000 L CNN
-F 1 "TL074" H 1558 5255 50  0000 L CNN
-F 2 "Package_DIP:DIP-14_W7.62mm_Socket" H 1550 5400 50  0001 C CNN
-F 3 "http://www.ti.com/lit/ds/symlink/tl071.pdf" H 1650 5500 50  0001 C CNN
-	5    1600 5300
+P 3225 4775
+F 0 "U1" H 3183 4821 50  0000 L CNN
+F 1 "TL074" H 3183 4730 50  0000 L CNN
+F 2 "Package_DIP:DIP-14_W7.62mm_Socket" H 3175 4875 50  0001 C CNN
+F 3 "http://www.ti.com/lit/ds/symlink/tl071.pdf" H 3275 4975 50  0001 C CNN
+	5    3225 4775
 	1    0    0    -1
 $EndComp
@@
 	2800 1675 2800 2325
 Connection ~ 2800 2325
-Text GLabel 2400 3725 0    50   Input ~ 0
-6V
+Text GLabel 2575 3725 0    50   Input ~ 0
+VREF
 Wire Wire Line
 	3975 3725 3975 3600
@@
 	2800 3725 3975 3725
 Wire Wire Line
-	2400 3725 2800 3725
+	2575 3725 2800 3725
 Wire Wire Line
 	3550 2775 3675 2775
@@
 Connection ~ 3675 2775
 Wire Wire Line
-	3675 2775 3675 4300
+	3675 2775 3675 4075
 NoConn ~ 12100 3000
 $Comp
 L power:+12V #PWR0106
 U 1 1 62957056
-P 1500 4825
-F 0 "#PWR0106" H 1500 4675 50  0001 C CNN
-F 1 "+12V" H 1515 4998 50  0000 C CNN
-F 2 "" H 1500 4825 50  0001 C CNN
-F 3 "" H 1500 4825 50  0001 C CNN
-	1    1500 4825
-	1    0    0    -1
-$EndComp
-Wire Wire Line
-	1500 5750 1500 5725
-Wire Wire Line
-	1500 5000 1500 4925
+P 3125 4300
+F 0 "#PWR0106" H 3125 4150 50  0001 C CNN
+F 1 "+12V" H 3140 4473 50  0000 C CNN
+F 2 "" H 3125 4300 50  0001 C CNN
+F 3 "" H 3125 4300 50  0001 C CNN
+	1    3125 4300
+	1    0    0    -1
+$EndComp
+Wire Wire Line
+	3125 5225 3125 5200
+Wire Wire Line
+	3125 4475 3125 4400
 Wire Wire Line
 	4150 3050 4125 3050
@@
 $EndComp
 Wire Wire Line
-	3675 4300 6175 4300
+	3675 4075 6175 4075
 $Comp
 L Switch:SW_DPDT_x2 SW1
@@
 $EndComp
 Wire Wire Line
-	6175 4300 6175 4550
+	6175 4075 6175 4550
 Wire Wire Line
 	6175 5100 6175 4850
@@
 	6825 3250 7600 3250
 Wire Wire Line
-	6150 3650 6150 3900
+	6150 3650 6150 3775
 Connection ~ 6150 3650
 Wire Wire Line
@@
 L power:GND #PWR0101
 U 1 1 62918B4B
-P 6150 3900
-F 0 "#PWR0101" H 6150 3650 50  0001 C CNN
-F 1 "GND" H 6155 3727 50  0000 C CNN
-F 2 "" H 6150 3900 50  0001 C CNN
-F 3 "" H 6150 3900 50  0001 C CNN
-	1    6150 3900
+P 6150 3775
+F 0 "#PWR0101" H 6150 3525 50  0001 C CNN
+F 1 "GND" H 6155 3602 50  0000 C CNN
+F 2 "" H 6150 3775 50  0001 C CNN
+F 3 "" H 6150 3775 50  0001 C CNN
+	1    6150 3775
 	1    0    0    -1
 $EndComp
@@
 L power:GND #PWR0107
 U 1 1 629A3B25
-P 1500 5750
-F 0 "#PWR0107" H 1500 5500 50  0001 C CNN
-F 1 "GND" H 1505 5577 50  0000 C CNN
-F 2 "" H 1500 5750 50  0001 C CNN
-F 3 "" H 1500 5750 50  0001 C CNN
-	1    1500 5750
+P 3125 5225
+F 0 "#PWR0107" H 3125 4975 50  0001 C CNN
+F 1 "GND" H 3130 5052 50  0000 C CNN
+F 2 "" H 3125 5225 50  0001 C CNN
+F 3 "" H 3125 5225 50  0001 C CNN
+	1    3125 5225
 	1    0    0    -1
 $EndComp
@@
 L Device:R R9
 U 1 1 629B7FF1
-P 1825 4925
-F 0 "R9" V 1725 4925 50  0000 C CNN
-F 1 "10K" V 1825 4925 50  0000 C CNN
-F 2 "benjiaomodular:Resistor_L6.3mm_D2.5mm_P7.62mm_Horizontal" V 1755 4925 50  0001 C CNN
-F 3 "~" H 1825 4925 50  0001 C CNN
-	1    1825 4925
+P 3450 4400
+F 0 "R9" V 3350 4400 50  0000 C CNN
+F 1 "10K" V 3450 4400 50  0000 C CNN
+F 2 "benjiaomodular:Resistor_L6.3mm_D2.5mm_P7.62mm_Horizontal" V 3380 4400 50  0001 C CNN
+F 3 "~" H 3450 4400 50  0001 C CNN
+	1    3450 4400
 	0    -1   -1   0
 $EndComp
@@
 L Device:R R10
 U 1 1 629B8C18
-P 2150 5225
-F 0 "R10" V 2050 5225 50  0000 C CNN
-F 1 "10K" V 2150 5225 50  0000 C CNN
-F 2 "benjiaomodular:Resistor_L6.3mm_D2.5mm_P7.62mm_Horizontal" V 2080 5225 50  0001 C CNN
-F 3 "~" H 2150 5225 50  0001 C CNN
-	1    2150 5225
-	1    0    0    -1
-$EndComp
-Wire Wire Line
-	1675 4925 1500 4925
-Connection ~ 1500 4925
-Wire Wire Line
-	1500 4925 1500 4850
-Wire Wire Line
-	1975 4925 2150 4925
-Wire Wire Line
-	2150 4925 2150 5075
-Wire Wire Line
-	2150 5375 2150 5650
-Wire Wire Line
-	2150 5650 1500 5650
-Connection ~ 1500 5650
-Wire Wire Line
-	1500 5650 1500 5600
-Text GLabel 2325 4925 2    50   Output ~ 0
-6V
-Wire Wire Line
-	2325 4925 2150 4925
-Connection ~ 2150 4925
+P 3775 4700
+F 0 "R10" V 3675 4700 50  0000 C CNN
+F 1 "10K" V 3775 4700 50  0000 C CNN
+F 2 "benjiaomodular:Resistor_L6.3mm_D2.5mm_P7.62mm_Horizontal" V 3705 4700 50  0001 C CNN
+F 3 "~" H 3775 4700 50  0001 C CNN
+	1    3775 4700
+	1    0    0    -1
+$EndComp
+Wire Wire Line
+	3300 4400 3125 4400
+Connection ~ 3125 4400
+Wire Wire Line
+	3125 4400 3125 4325
+Wire Wire Line
+	3600 4400 3775 4400
+Wire Wire Line
+	3775 4400 3775 4550
+Wire Wire Line
+	3775 4850 3775 5125
+Wire Wire Line
+	3775 5125 3125 5125
+Connection ~ 3125 5125
+Wire Wire Line
+	3125 5125 3125 5075
+Text GLabel 3950 4400 2    50   Output ~ 0
+VREF
+Wire Wire Line
+	3950 4400 3775 4400
+Connection ~ 3775 4400
 $Comp
 L power:PWR_FLAG #FLG0101
 U 1 1 629D9F93
-P 1500 4850
-F 0 "#FLG0101" H 1500 4925 50  0001 C CNN
-F 1 "PWR_FLAG" V 1500 4977 50  0000 L CNN
-F 2 "" H 1500 4850 50  0001 C CNN
-F 3 "~" H 1500 4850 50  0001 C CNN
-	1    1500 4850
+P 3125 4325
+F 0 "#FLG0101" H 3125 4400 50  0001 C CNN
+F 1 "PWR_FLAG" V 3125 4452 50  0000 L CNN
+F 2 "" H 3125 4325 50  0001 C CNN
+F 3 "~" H 3125 4325 50  0001 C CNN
+	1    3125 4325
 	0    -1   -1   0
 $EndComp
-Connection ~ 1500 4850
-Wire Wire Line
-	1500 4850 1500 4825
+Connection ~ 3125 4325
+Wire Wire Line
+	3125 4325 3125 4300
 $Comp
 L power:PWR_FLAG #FLG0102
 U 1 1 629DB4AB
-P 1500 5725
-F 0 "#FLG0102" H 1500 5800 50  0001 C CNN
-F 1 "PWR_FLAG" V 1500 5852 50  0000 L CNN
-F 2 "" H 1500 5725 50  0001 C CNN
-F 3 "~" H 1500 5725 50  0001 C CNN
-	1    1500 5725
+P 3125 5200
+F 0 "#FLG0102" H 3125 5275 50  0001 C CNN
+F 1 "PWR_FLAG" V 3125 5327 50  0000 L CNN
+F 2 "" H 3125 5200 50  0001 C CNN
+F 3 "~" H 3125 5200 50  0001 C CNN
+	1    3125 5200
 	0    -1   -1   0
 $EndComp
-Connection ~ 1500 5725
-Wire Wire Line
-	1500 5725 1500 5650
+Connection ~ 3125 5200
+Wire Wire Line
+	3125 5200 3125 5125
 $EndSCHEMATC
